File: Ethernet.kicad_sch (KiCad schematic)
At the start: 34 parts, among them J2 ARJM11C7-009-AB-EW2, U3 LAN8742A, U4 USBLC6-4SC6, Y1 25Mhz

Commit message: Se estandariza algunos atributos: valores, librerias. Se actualiza pcb y se guarda.
Parts:
- C28: footprint 1-Capacitor:C_0603_1608Metric -> Capacitor_SMD:C_0805_2012Metric
- C29: value 1uF 16V -> 1uF/50V; footprint 1-Capacitor:C_0603_1608Metric -> Capacitor_SMD:C_0805_2012Metric
- C34, C38: value 100nF 50V -> 100nF/50V
- C35, C37: value 100nF 50V -> 100nF/50V; footprint 1-Capacitor:C_0805_2012Metric -> 1-Capacitor:C_0603_1608Metric
- R26: value 1k5 -> 1k
Changed lines of the file:
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@@
 			)
 		)
-		(property "Value" "100nF 50V"
+		(property "Value" "100nF/50V"
 			(at 239.014 81.28 0)
 			(effects
@@
 			)
 		)
-		(property "Value" "1k5"
+		(property "Value" "1k"
 			(at 91.948 87.376 0)
 			(effects
@@
 			)
 		)
-		(property "Footprint" "1-Capacitor:C_0603_1608Metric"
+		(property "Footprint" "Capacitor_SMD:C_0805_2012Metric"
 			(at 150.1648 41.91 0)
 			(effects
@@
 			)
 		)
-		(property "Value" "100nF 50V"
+		(property "Value" "100nF/50V"
 			(at 172.466 142.24 0)
 			(effects
@@
 			)
 		)
-		(property "Footprint" "1-Capacitor:C_0805_2012Metric"
+		(property "Footprint" "1-Capacitor:C_0603_1608Metric"
 			(at 174.2948 144.78 0)
 			(effects
@@
 			)
 		)
-		(property "Value" "100nF 50V"
+		(property "Value" "100nF/50V"
 			(at 185.674 142.24 0)
 			(effects
@@
 			)
 		)
-		(property "Footprint" "1-Capacitor:C_0805_2012Metric"
+		(property "Footprint" "1-Capacitor:C_0603_1608Metric"
 			(at 183.8452 144.78 0)
 			(effects
@@
 			)
 		)
-		(property "Value" "100nF 50V"
+		(property "Value" "100nF/50V"
 			(at 120.396 64.77 0)
 			(effects
@@
 			)
 		)
-		(property "Value" "1uF 16V"
+		(property "Value" "1uF/50V"
 			(at 103.886 39.37 0)
 			(effects
@@
 			)
 		)
-		(property "Footprint" "1-Capacitor:C_0603_1608Metric"
+		(property "Footprint" "Capacitor_SMD:C_0805_2012Metric"
 			(at 105.7148 41.91 0)
 			(effects

Commit message: Se estandariza losc omponentes, se cambian algunos valores para evitar gastos adicionales. Se termina y comprueb el part list para jlcpcb
Parts:
- FB2: value 600R -> 450mR/200mA; footprint Inductor_SMD:L_0805_2012Metric -> Inductor_SMD:L_0603_1608Metric
- R27, R28: value 510R -> 10k
Changed lines of the file:
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@@
 	(text "C1002"
 		(exclude_from_sim no)
-		(at 191.77 40.894 0)
+		(at 191.008 35.56 0)
 		(effects
 			(font
@@
 			)
 		)
-		(property "Value" "510R"
+		(property "Value" "10k"
 			(at 253.238 144.526 0)
 			(effects
@@
 		(dnp no)
 		(property "Reference" "FB2"
-			(at 189.992 26.416 90)
+			(at 183.388 26.924 90)
 			(effects
 				(font
@@
 			)
 		)
-		(property "Value" "600R"
-			(at 189.992 28.956 90)
+		(property "Value" "450mR/200mA"
+			(at 188.722 28.956 90)
 			(effects
 				(font
@@
 			)
 		)
-		(property "Footprint" "Inductor_SMD:L_0805_2012Metric"
+		(property "Footprint" "Inductor_SMD:L_0603_1608Metric"
 			(at 190.5 33.528 90)
 			(effects
@@
 			)
 		)
-		(property "Value" "510R"
+		(property "Value" "10k"
 			(at 275.082 144.526 0)
 			(effects
