File: Serial.kicad_sch (KiCad schematic)
At the start: 21 parts, among them J42 DE9_Receptacle_MountingHoles, J45 USB_A_Female_P2.5mm, U11 USBLC6-2SC6, U14 MAX232

Commit message: Se estandariza algunos atributos: valores, librerias. Se actualiza pcb y se guarda.
Parts:
- C69, C73: value 100nF 50V -> 100nF/50V; footprint 1-Capacitor:C_0805_2012Metric -> 1-Capacitor:C_0603_1608Metric
- C70, C71, C72, C74: value 1uF 50V -> 1uF/50V; footprint 1-Capacitor:C_0805_2012Metric -> Capacitor_SMD:C_0805_2012Metric
Changed lines of the file:
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@@
 			)
 		)
-		(property "Value" "100nF 50V"
+		(property "Value" "100nF/50V"
 			(at 57.15 44.4499 0)
 			(effects
@@
 			)
 		)
-		(property "Footprint" "1-Capacitor:C_0805_2012Metric"
+		(property "Footprint" "1-Capacitor:C_0603_1608Metric"
 			(at 54.3052 46.99 0)
 			(effects
@@
 			)
 		)
-		(property "Value" "1uF 50V"
+		(property "Value" "1uF/50V"
 			(at 140.97 43.18 0)
 			(effects
@@
 			)
 		)
-		(property "Footprint" "1-Capacitor:C_0805_2012Metric"
+		(property "Footprint" "Capacitor_SMD:C_0805_2012Metric"
 			(at 138.1252 45.72 0)
 			(effects
@@
 			)
 		)
-		(property "Value" "1uF 50V"
+		(property "Value" "1uF/50V"
 			(at 73.66 44.45 0)
 			(effects
@@
 			)
 		)
-		(property "Footprint" "1-Capacitor:C_0805_2012Metric"
+		(property "Footprint" "Capacitor_SMD:C_0805_2012Metric"
 			(at 87.3252 45.72 0)
 			(effects
@@
 			)
 		)
-		(property "Value" "100nF 50V"
+		(property "Value" "100nF/50V"
 			(at 121.92 133.3499 0)
 			(effects
@@
 			)
 		)
-		(property "Footprint" "1-Capacitor:C_0805_2012Metric"
+		(property "Footprint" "1-Capacitor:C_0603_1608Metric"
 			(at 124.7648 135.89 0)
 			(effects
@@
 			)
 		)
-		(property "Value" "1uF 50V"
+		(property "Value" "1uF/50V"
 			(at 176.53 57.15 0)
 			(effects
@@
 			)
 		)
-		(property "Footprint" "1-Capacitor:C_0805_2012Metric"
+		(property "Footprint" "Capacitor_SMD:C_0805_2012Metric"
 			(at 162.8648 58.42 0)
 			(effects
@@
 			)
 		)
-		(property "Value" "1uF 50V"
+		(property "Value" "1uF/50V"
 			(at 157.48 59.69 0)
 			(effects
@@
 			)
 		)
-		(property "Footprint" "1-Capacitor:C_0805_2012Metric"
+		(property "Footprint" "Capacitor_SMD:C_0805_2012Metric"
 			(at 146.3548 60.96 0)
 			(effects

Commit message: Se estandariza losc omponentes, se cambian algunos valores para evitar gastos adicionales. Se termina y comprueb el part list para jlcpcb
Parts:
- R225: value 2k -> 20k
- R226, R227, R70: value 1k -> 10k
Changed lines of the file:
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@@
 			)
 		)
-		(property "Value" "2k"
+		(property "Value" "20k"
 			(at 30.48 81.28 0)
 			(effects
@@
 			)
 		)
-		(property "Value" "1k"
+		(property "Value" "10k"
 			(at 50.8 82.55 90)
 			(effects
@@
 			)
 		)
-		(property "Value" "1k"
+		(property "Value" "10k"
 			(at 41.91 76.2 90)
 			(effects
@@
 			)
 		)
-		(property "Value" "1k"
+		(property "Value" "10k"
 			(at 58.42 82.55 90)
 			(effects

Commit message: Se añade led status y eeprom externa. Se actutliza y añade serigrafía a la pcb, se escoge uC de menos flash debido a la escasez del uC planeado, sin embargo, funcionará a recomendacion del programador. Se revisa en jlcpcb y se espera su envío
Connections:
- no-connect marks 0 -> 8
Changed lines of the file:
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@@
 		(color 0 0 0 0)
+	)
+	(no_connect
+		(at 91.44 78.74)
+	)
+	(no_connect
+		(at 91.44 68.58)
+	)
+	(no_connect
+		(at 195.58 44.45)
+	)
+	(no_connect
+		(at 195.58 36.83)
+	)
+	(no_connect
+		(at 195.58 31.75)
+	)
+	(no_connect
+		(at 195.58 46.99)
+	)
+	(no_connect
+		(at 195.58 41.91)
+	)
+	(no_connect
+		(at 195.58 29.21)
 	)
 	(wire
